File: KiCAD/rover-electronics/rover-electronics.kicad_sch (KiCad schematic)
At the start: 23 parts, among them M1 Stepper_Motor_bipolar, M2 Stepper_Motor_bipolar, M3 Stepper_Motor_bipolar, M4 Motor_DC, M5 Motor_DC, M6 Motor_DC, M7 Motor_DC, M8 Motor_DC, M9 Motor_DC, U1 DRV8871DDA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

Commit message: Minor fixes for Schematics
Connections:
- net +12V: no longer RPi-4b1. (USB_C_GND)
- net at U7.2 (OUT): now also RPi-4b1. (USB_C_GND)
- net at RPi-4b1.23 (GPIO_11): now also ULM1. (Out4)
- net at RPi-4b1.29 (GPIO_5): now also ULM1. (Out4)
- net at RPi-4b1.31 (GPIO_6): now also ULM1. (Out4)
- net at RPi-4b1.33 (GPIO_13): now also ULM1. (Out4)
Changed lines of the file:
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@@
-	)
-	(junction
-		(at 73.66 101.6)
-		(diameter 0)
-		(color 0 0 0 0)
 	)
 	(junction
@@
 	(wire
 		(pts
+			(xy 137.16 55.88) (xy 137.16 106.68)
+		)
+		(stroke
+			(width 0)
+			(type default)
+		)
+	)
+	(wire
+		(pts
 			(xy 160.02 153.67) (xy 146.05 153.67)
 		)
@@
 	(wire
 		(pts
-			(xy 73.66 101.6) (xy 95.25 101.6)
-		)
-		(stroke
-			(width 0)
-			(type default)
-		)
-	)
-	(wire
-		(pts
-			(xy 73.66 125.73) (xy 73.66 101.6)
+			(xy 73.66 96.52) (xy 73.66 125.73)
 		)
 		(stroke
@@
 	(wire
 		(pts
+			(xy 151.13 53.34) (xy 135.89 53.34)
+		)
+		(stroke
+			(width 0)
+			(type default)
+		)
+	)
+	(wire
+		(pts
 			(xy 172.72 109.22) (xy 186.69 109.22)
 		)
@@
 	(wire
 		(pts
+			(xy 151.13 63.5) (xy 139.7 63.5)
+		)
+		(stroke
+			(width 0)
+			(type default)
+		)
+	)
+	(wire
+		(pts
 			(xy 186.69 149.86) (xy 182.88 149.86)
 		)
@@
 	(wire
 		(pts
+			(xy 137.16 106.68) (xy 130.81 106.68)
+		)
+		(stroke
+			(width 0)
+			(type default)
+		)
+	)
+	(wire
+		(pts
 			(xy 180.34 87.63) (xy 170.18 87.63)
 		)
@@
 	(wire
 		(pts
+			(xy 151.13 55.88) (xy 137.16 55.88)
+		)
+		(stroke
+			(width 0)
+			(type default)
+		)
+	)
+	(wire
+		(pts
 			(xy 99.06 154.94) (xy 99.06 158.75)
 		)
@@
 	(wire
 		(pts
+			(xy 135.89 104.14) (xy 130.81 104.14)
+		)
+		(stroke
+			(width 0)
+			(type default)
+		)
+	)
+	(wire
+		(pts
 			(xy 148.59 152.4) (xy 160.02 152.4)
 		)
@@
 	(wire
 		(pts
+			(xy 138.43 109.22) (xy 130.81 109.22)
+		)
+		(stroke
+			(width 0)
+			(type default)
+		)
+	)
+	(wire
+		(pts
 			(xy 60.96 107.95) (xy 72.39 107.95)
 		)
@@
 	(wire
 		(pts
+			(xy 93.98 101.6) (xy 95.25 101.6)
+		)
+		(stroke
+			(width 0)
+			(type default)
+		)
+	)
+	(wire
+		(pts
 			(xy 71.12 91.44) (xy 80.01 91.44)
 		)
@@
 	(wire
 		(pts
+			(xy 138.43 60.96) (xy 138.43 109.22)
+		)
+		(stroke
+			(width 0)
+			(type default)
+		)
+	)
+	(wire
+		(pts
 			(xy 143.51 111.76) (xy 149.86 111.76)
 		)
@@
 	(wire
 		(pts
+			(xy 93.98 81.28) (xy 93.98 101.6)
+		)
+		(stroke
+			(width 0)
+			(type default)
+		)
+	)
+	(wire
+		(pts
 			(xy 60.96 151.13) (xy 73.66 151.13)
 		)
@@
 	(wire
 		(pts
+			(xy 139.7 63.5) (xy 139.7 114.3)
+		)
+		(stroke
+			(width 0)
+			(type default)
+		)
+	)
+	(wire
+		(pts
 			(xy 139.7 180.34) (xy 139.7 189.23)
 		)
@@
 	(wire
 		(pts
-			(xy 73.66 101.6) (xy 73.66 96.52)
-		)
-		(stroke
-			(width 0)
-			(type default)
-		)
-	)
-	(wire
-		(pts
 			(xy 134.62 154.94) (xy 132.08 154.94)
 		)
@@
 	(wire
 		(pts
+			(xy 151.13 60.96) (xy 138.43 60.96)
+		)
+		(stroke
+			(width 0)
+			(type default)
+		)
+	)
+	(wire
+		(pts
 			(xy 140.97 77.47) (xy 140.97 83.82)
 		)
@@
 	(wire
 		(pts
+			(xy 125.73 81.28) (xy 93.98 81.28)
+		)
+		(stroke
+			(width 0)
+			(type default)
+		)
+	)
+	(wire
+		(pts
 			(xy 45.72 71.12) (xy 45.72 54.61)
 		)
@@
 	(wire
 		(pts
+			(xy 139.7 114.3) (xy 130.81 114.3)
+		)
+		(stroke
+			(width 0)
+			(type default)
+		)
+	)
+	(wire
+		(pts
 			(xy 160.02 77.47) (xy 160.02 67.31)
 		)
@@
 		)
 		(stroke
+			(width 0)
+			(type default)
+		)
+	)
+	(wire
+		(pts
+			(xy 135.89 53.34) (xy 135.89 104.14)
+		)
+		(stroke
